Commit message: ros2_tutorials course2 FinalProj part1 robotic_arm

File: src/my_robot_description/urdf/Course2_Actv01.xacro (robot description, xacro)
@@ -6,8 +6,17 @@
     <xacro:property name="wheel_radius" value="0.1" />
     <xacro:property name="wheel_length" value="0.05" />
+    <xacro:property name="arm_base_length" value="0.1"/>
+    <xacro:property name="arm_base_width" value="0.1"/>
+    <xacro:property name="arm_base_height" value="0.02"/>
+    <xacro:property name="forearm_radius" value="0.02" />
+    <xacro:property name="forearm_length" value="0.3" />
+    <xacro:property name="hand_radius" value="0.02" />
+    <xacro:property name="hand_length" value="0.3" />
     <xacro:include filename="common_properties.xacro"/>
-    <xacro:include filename="mobile_base.xacro"/>
+    <!-- <xacro:include filename="mobile_base.xacro"/>
     <xacro:include filename="mobile_base_gazebo.xacro"/>
-    <xacro:include filename="camera.xacro"/>
+    <xacro:include filename="camera.xacro"/> -->
+    <xacro:include filename="ros2_L2_finalproj_Arm.xacro"/>
+    <xacro:include filename="ros2_L2_finalproj_Arm_gazebo.xacro"/>
 </robot>
 <!-- THIS PART IS COMMENTED OUT TO DEMONSTRATE THE USAGE OF XACRO INSIDE ANOTHER XACRO

File: src/my_robot_description/urdf/common_properties.xacro (robot description, xacro)
@@ -2,11 +2,17 @@
 <robot xmlns:xacro="http://www.ros.org/wiki/xacro">
     <material name="blue">
-        <color rgba="1 0 0 1"/>
+        <color rgba="0 0 1 1"/>
     </material>
     <material name="grey">
-        <color rgba="0 0 1 1"/>
+        <color rgba="0.5 0.5 0.5 1"/>
     </material>
     <material name="black">
-    <color rgba="1 1 1 1"/>
+        <color rgba="0 0 0 1"/>
+    </material>
+    <material name="orange">
+        <color rgba="1 0.5 0 1"/>
+    </material>
+    <material name="yellow">
+        <color rgba="1 1 0 1"/>
     </material>
     <xacro:macro name="box_inertia" params="m x y z o_xyz o_rpy">
@@ -28,4 +34,22 @@
         </inertial>
     </xacro:macro>
+    <xacro:macro name="forearm_inertia" params="m r h o_xyz o_rpy">
+        <inertial>
+            <mass value="${m}" />
+            <origin xyz="${o_xyz}" rpy="${o_rpy}" />
+            <inertia ixx="${(m/12)*(3*r*r + h*h)}" ixy="0" ixz="0"
+                     iyy="${(m/12)*(3*r*r + h*h)}" iyz="0"
+                     izz="${0.5*m*r*r}"/>
+        </inertial>
+    </xacro:macro>
+    <xacro:macro name="hand_inertia" params="m r h o_xyz o_rpy">
+        <inertial>
+            <mass value="${m}" />
+            <origin xyz="${o_xyz}" rpy="${o_rpy}" />
+            <inertia ixx="${(m/12)*(3*r*r + h*h)}" ixy="0" ixz="0"
+                     iyy="${(m/12)*(3*r*r + h*h)}" iyz="0"
+                     izz="${0.5*m*r*r}"/>
+        </inertial>
+    </xacro:macro>
     <xacro:macro name="caster_wheel_inertia" params="m r o_xyz o_rpy">
         <inertial>

Commit message: ros2_tutorials course2 FinalProj part2 robotic_arm on robot_base

File: src/my_robot_description/urdf/Course2_Actv01.xacro (robot description, xacro)
@@ -14,7 +14,7 @@
     <xacro:property name="hand_length" value="0.3" />
     <xacro:include filename="common_properties.xacro"/>
-    <!-- <xacro:include filename="mobile_base.xacro"/>
+    <xacro:include filename="mobile_base.xacro"/>
     <xacro:include filename="mobile_base_gazebo.xacro"/>
-    <xacro:include filename="camera.xacro"/> -->
+    <xacro:include filename="camera.xacro"/>
     <xacro:include filename="ros2_L2_finalproj_Arm.xacro"/>
     <xacro:include filename="ros2_L2_finalproj_Arm_gazebo.xacro"/>

File: src/my_robot_description/urdf/ros2_L2_finalproj_Arm.xacro (robot description, xacro)
@@ -65,3 +65,8 @@
         <dynamics damping="0.3" friction="0.3"/>
     </joint>
+    <joint name="base_arm_joint" type="fixed">
+        <parent link="base_link"/>
+        <child link="arm_base_link"/>
+        <origin xyz="${base_length/3.0} 0 ${base_height}" rpy="0 0 0"/>
+    </joint>
 </robot>
