Commit message: ros2_tutorials course2 FinalProj joint _state_publisher and inertia pos correction

File: src/my_robot_description/urdf/ros2_L2_finalproj_Arm.xacro (robot description, xacro)
@@ -22,8 +22,8 @@
                     <cylinder radius="${forearm_radius}" length="${forearm_length}"/>
                 </geometry>
-                <origin xyz="0 0 ${(forearm_length)/2}" rpy="0 0 0"/>
+                <origin xyz="0 0 ${forearm_length/2}" rpy="0 0 0"/>
                 <material name="yellow"/>
             </visual>
-            <xacro:forearm_inertia m="0.3" r="${forearm_radius}" h="${forearm_length}" o_xyz="0 0 0" o_rpy="0 0 0" />
+            <xacro:forearm_inertia m="0.3" r="${forearm_radius}" h="${forearm_length}" o_xyz="0 0 ${forearm_length/2}" o_rpy="0 0 0" />
             <collision>
                 <geometry>
@@ -41,5 +41,5 @@
                 <material name="orange"/>
             </visual>
-            <xacro:hand_inertia m="0.3" r="${hand_radius}" h="${hand_length}" o_xyz="0 0 0" o_rpy="0 0 0" />
+            <xacro:hand_inertia m="0.3" r="${hand_radius}" h="${hand_length}" o_xyz="0 0 ${forearm_length/2}" o_rpy="0 0 0" />
             <collision>
                 <geometry>

File: src/my_robot_description/urdf/ros2_L2_finalproj_Arm_gazebo.xacro (robot description, xacro)
@@ -23,3 +23,11 @@
         </plugin>
     </gazebo>
+    <gazebo>
+        <plugin
+            filename="gz-sim-joint-state-publisher-system"
+            name="gz::sim::systems::JointStatePublisher">
+            <joint_name>arm_base_forearm_joint</joint_name>
+            <joint_name>forearm_hand_joint</joint_name>
+        </plugin>
+    </gazebo>
 </robot>
