Commit message: ros2_tutorials Ackermann controller controller config and launch file

File: src/my_robot_description/urdf/Ackermann_robot_model.xacro (robot description, xacro)
@@ -10,5 +10,5 @@
   <!-- ================= PARAMETERS ================= -->
   <!--
-    Coordinate convention:
+    Coordinate convention
       X = Forward
       Y = Left
@@ -78,5 +78,5 @@
     <parent link="rear_left_rack_support_link"/>
     <child link="rear_left_wheel"/>
-    <origin xyz="0 0 ${-wheel_length}" rpy="1.57 0 0"/>
+    <origin xyz="0 0 ${-wheel_length}" rpy="-1.57 0 0"/>
     <axis xyz="0 1 0"/>
     <dynamics damping="0.1"/>
@@ -116,5 +116,5 @@
     <parent link="rear_right_rack_support_link"/>
     <child link="rear_right_wheel"/>
-    <origin xyz="0 0 ${wheel_length}" rpy="1.57 0 0"/>
+    <origin xyz="0 0 ${wheel_length}" rpy="-1.57 0 0"/>
     <axis xyz="0 1 0"/>
     <dynamics damping="0.1"/>
@@ -148,5 +148,5 @@
     <parent link="front_left_rack_support_link"/>
     <child link="front_left_steering_support_link"/>
-    <origin xyz="0 0 ${-base_width/4}" rpy="${pi/2} 0 0"/>
+    <origin xyz="0 0 ${-base_width/4}" rpy="${-pi/2} 0 0"/>
     <axis xyz="0 0 1"/>
     <limit
@@ -177,5 +177,5 @@
     <child link="front_left_wheel"/>
     <origin xyz="0 0 0" rpy="0 ${pi/2} 0"/>
-    <axis xyz="0 1 0"/>
+    <axis xyz="0 -1 0"/>
     <dynamics damping="0.1"/>
   </joint>
@@ -208,5 +208,5 @@
     <parent link="front_right_rack_support_link"/>
     <child link="front_right_steering_support_link"/>
-    <origin xyz="0 0 ${base_width/4}" rpy="${pi/2} 0 0"/>
+    <origin xyz="0 0 ${base_width/4}" rpy="${-pi/2} 0 0"/>
     <axis xyz="0 0 1"/>
     <limit
@@ -237,9 +237,9 @@
     <child link="front_right_wheel"/>
     <origin xyz="0 0 0" rpy="0 ${pi/2} 0"/>
-    <axis xyz="0 1 0"/>
+    <axis xyz="0 -1 0"/>
     <dynamics damping="0.1"/>
   </joint>
   <!-- ================= ROS 2 CONTROL ================= -->
-  <ros2_control name="GazeboSimSystem" type="system">
+  <ros2_control name="AckermannRobotSystem" type="system">
     <hardware>
       <plugin>gz_ros2_control/GazeboSimSystem</plugin>
@@ -283,5 +283,5 @@
       name="gz_ros2_control::GazeboSimROS2ControlPlugin">
       <parameters>
-        $(find ackermann_robot_description)/config/ackermann_controller.yaml
+        $(find my_ros2_bringup)/config/ackermann_controller.yaml
       </parameters>
     </plugin>

Commit message: ros2_tutorials Ackermann robot chasis size reduced

File: src/my_robot_description/urdf/Ackermann_robot_model.xacro (robot description, xacro)
@@ -2,5 +2,5 @@
 <robot name="ackermann_robot" xmlns:xacro="http://www.ros.org/wiki/xacro">
     <xacro:include filename="common_properties.xacro"/>
-    <xacro:property name="base_length" value="1.2" />
+    <xacro:property name="base_length" value="0.8" />
     <xacro:property name="base_width" value="0.35" />
     <xacro:property name="base_height" value="0.2" />
@@ -14,5 +14,5 @@
       Y = Left
       Z = Up
-    Wheelbase = 1.0 m
+    Wheelbase = 0.7 m
     Track width = 0.6 m
     Wheel radius = 0.15 m
@@ -35,5 +35,5 @@
       <origin xyz="0 0 0.1" rpy="0 0 0"/>
     </collision>
-    <xacro:box_inertia m="15.0" x="1.2" y="0.5" z="0.2" o_xyz="0 0 0" o_rpy="0 0 0" />
+    <xacro:box_inertia m="15.0" x="${base_length}" y="${base_width}" z="${base_height}" o_xyz="0 0 0" o_rpy="0 0 0" />
   </link>
   <link name="base_footprint_link"/>
@@ -57,5 +57,5 @@
     <parent link="base_link"/>
     <child link="rear_left_rack_support_link"/>
-    <origin xyz="-0.5 ${(base_width/2)+0.05} 0" rpy="${pi/2} 0 0"/>
+    <origin xyz="${-base_length/2 + 0.05} ${(base_width/2)+0.05} 0" rpy="${pi/2} 0 0"/>
   </joint>
   <!-- ================= REAR LEFT WHEEL ================= -->
@@ -95,5 +95,5 @@
     <parent link="base_link"/>
     <child link="rear_right_rack_support_link"/>
-    <origin xyz="-0.5 ${-(base_width/2)-0.05} 0" rpy="${pi/2} 0 0"/>
+    <origin xyz="${-base_length/2 + 0.05} ${-(base_width/2)-0.05} 0" rpy="${pi/2} 0 0"/>
   </joint>
   <!-- ================= REAR RIGHT WHEEL ================= -->
@@ -133,5 +133,5 @@
     <parent link="base_link"/>
     <child link="front_left_rack_support_link"/>
-    <origin xyz="0.5 ${(base_width/2)+0.05} 0" rpy="${pi/2} 0 0"/>
+    <origin xyz="${base_length/2 - 0.05} ${(base_width/2)+0.05} 0" rpy="${pi/2} 0 0"/>
   </joint>
   <!-- ================= FRONT LEFT STEERING SUPPORT================= -->
@@ -193,5 +193,5 @@
     <parent link="base_link"/>
     <child link="front_right_rack_support_link"/>
-    <origin xyz="0.5 ${-(base_width/2)-0.05} 0" rpy="${pi/2} 0 0"/>
+    <origin xyz="${base_length/2 - 0.05} ${-(base_width/2)-0.05} 0" rpy="${pi/2} 0 0"/>
   </joint>
   <!-- ================= FRONT RIGHT STEERING SUPPORT================= -->

Commit message: ros2_tutorials Ackermann robot dimensions updated to achive 1m turning radius

File: src/my_robot_description/urdf/Ackermann_robot_model.xacro (robot description, xacro)
@@ -2,6 +2,6 @@
 <robot name="ackermann_robot" xmlns:xacro="http://www.ros.org/wiki/xacro">
     <xacro:include filename="common_properties.xacro"/>
-    <xacro:property name="base_length" value="0.8" />
-    <xacro:property name="base_width" value="0.35" />
+    <xacro:property name="base_length" value="0.6" />
+    <xacro:property name="base_width" value="0.30" />
     <xacro:property name="base_height" value="0.2" />
     <xacro:property name="wheel_radius" value="0.15" />
@@ -14,6 +14,7 @@
       Y = Left
       Z = Up
-    Wheelbase = 0.7 m
-    Track width = 0.6 m
+    Wheelbase = 0.50 m
+    Front steering track width = 0.55 m
+    Rear traction track width = 0.56 m
     Wheel radius = 0.15 m
   -->
