Commit message: ros2_tutorials AGV renaming - common prop adaptations - camera integration

File: src/my_robot_description/urdf/AGV_model.xacro (robot description, xacro)
@@ -1,10 +1,6 @@
 <?xml version="1.0"?>
-<robot name="ackermann_robot" xmlns:xacro="http://www.ros.org/wiki/xacro">
-    <xacro:include filename="common_properties.xacro"/>
-    <xacro:property name="base_length" value="0.6" />
-    <xacro:property name="base_width" value="0.30" />
-    <xacro:property name="base_height" value="0.2" />
-    <xacro:property name="wheel_radius" value="0.15" />
-    <xacro:property name="wheel_length" value="0.08" />
+<robot name="AGV" xmlns:xacro="http://www.ros.org/wiki/xacro">
+    <xacro:include filename="AGV_common_properties.xacro"/>
+    <xacro:include filename="AGV_camera.xacro"/>
     <!-- <xacro:property name="pi" value="3.14159" /> -->
   <!-- ================= PARAMETERS ================= -->
@@ -25,7 +21,5 @@
         <box size="${base_length} ${base_width} ${base_height}"/>
       </geometry>
-      <material name="blue">
-        <color rgba="0.1 0.3 0.8 1.0"/>
-      </material>
+      <material name="AGV_blue"/>
       <origin xyz="0 0 0.1" rpy="0 0 0"/>
     </visual>
@@ -51,5 +45,5 @@
         <cylinder radius="0.01" length="${base_width/2}"/>
       </geometry>
-      <material name="black"/>
+      <material name="AGV_black"/>
     </visual>
     <xacro:wheel_inertia m="1.0" r="0.01" h="${base_width/2}" o_xyz="0 0 0" o_rpy="0 0 0" />
@@ -89,5 +83,5 @@
         <cylinder radius="0.01" length="${base_width/2}"/>
       </geometry>
-      <material name="black"/>
+      <material name="AGV_black"/>
     </visual>
     <xacro:wheel_inertia m="1.0" r="0.01" h="${base_width/2}" o_xyz="0 0 0" o_rpy="0 0 0" />
@@ -127,5 +121,5 @@
         <cylinder radius="0.01" length="${base_width/2}"/>
       </geometry>
-      <material name="black"/>
+      <material name="AGV_black"/>
     </visual>
     <xacro:wheel_inertia m="1.0" r="0.01" h="${base_width/2}" o_xyz="0 0 0" o_rpy="0 0 0" />
@@ -142,5 +136,5 @@
         <cylinder radius="0.015" length="${base_width/6}"/>
       </geometry>
-      <material name="grey"/>
+      <material name="AGV_grey"/>
     </visual>
     <xacro:wheel_inertia m="1.0" r="0.02" h="${base_width/4}" o_xyz="0 0 0" o_rpy="0 0 0" />
@@ -187,5 +181,5 @@
         <cylinder radius="0.01" length="${base_width/2}"/>
       </geometry>
-      <material name="black"/>
+      <material name="AGV_black"/>
     </visual>
     <xacro:wheel_inertia m="1.0" r="0.01" h="${base_width/2}" o_xyz="0 0 0" o_rpy="0 0 0" />
@@ -202,5 +196,5 @@
         <cylinder radius="0.015" length="${base_width/6}"/>
       </geometry>
-      <material name="grey"/>
+      <material name="AGV_grey"/>
     </visual>
     <xacro:wheel_inertia m="1.0" r="0.02" h="${base_width/4}" o_xyz="0 0 0" o_rpy="0 0 0" />
