Commit message: ros2_tutorials AGV Proper camera adaptations

File: src/my_robot_description/urdf/AGV_camera.xacro (robot description, xacro)
@@ -1,6 +1,6 @@
 <?xml version="1.0"?>
 <robot xmlns:xacro="http://www.ros.org/wiki/xacro">
-    <xacro:property name="camera_length" value="0.1"/>
-    <xacro:property name="camera_width" value="0.01"/>
+    <xacro:property name="camera_length" value="0.01"/>
+    <xacro:property name="camera_width" value="0.1"/>
     <xacro:property name="camera_height" value="0.025"/>
     <link name="camera_link">
@@ -21,9 +21,9 @@
         <parent link="base_link"/>
         <child link="camera_link"/>
-        <origin xyz="${(base_length+camera_width)/2} 0 ${base_height-(camera_height/2)}" rpy="0 0 ${-pi/2}"/>
+        <origin xyz="${(base_length+camera_length)/2} 0 ${base_height-(camera_height/2)}" rpy="0 0 0"/>
     </joint>
     <link name="camera_link_optical" />
     <joint name="camera_optical_joint" type="fixed">
-        <origin xyz="0 0 0" rpy="${-pi/2} 0 ${-pi/2}"/>
+        <origin xyz="0 0 0" rpy="0 ${-pi/2} 0"/>
         <parent link="camera_link"/>
         <child link="camera_link_optical"/>
