Commit message: ros2_tutorials AGV Wheel size reduced

File: src/my_robot_description/urdf/AGV_common_properties.xacro (robot description, xacro)
@@ -4,5 +4,5 @@
     <xacro:property name="base_width" value="0.30" />
     <xacro:property name="base_height" value="0.2" />
-    <xacro:property name="wheel_radius" value="0.15" />
+    <xacro:property name="wheel_radius" value="0.12" />
     <xacro:property name="wheel_length" value="0.08" />
     <material name="AGV_blue">

File: src/my_robot_description/urdf/AGV_model.xacro (robot description, xacro)
@@ -37,5 +37,5 @@
         <parent link="base_footprint_link"/>
         <child link="base_link"/>
-        <origin xyz="0 0 0.15" rpy="0 0 0"/>
+        <origin xyz="0 0 0.12" rpy="0 0 0"/>
         <axis xyz="0 0 0" />
   </joint>
@@ -69,5 +69,5 @@
       </geometry>
     </collision>
-    <xacro:wheel_inertia m="1.0" r="0.15" h="0.08" o_xyz="0 0 0" o_rpy="1.5707963 0 0" />
+    <xacro:wheel_inertia m="1.0" r="${wheel_radius}" h="${wheel_length}" o_xyz="0 0 0" o_rpy="1.5707963 0 0" />
   </link>
   <joint name="rear_left_rack_wheel_joint" type="continuous">
@@ -107,5 +107,5 @@
       </geometry>
     </collision>
-    <xacro:wheel_inertia m="1.0" r="0.15" h="0.08" o_xyz="0 0 0" o_rpy="1.5707963 0 0" />
+    <xacro:wheel_inertia m="1.0" r="${wheel_radius}" h="${wheel_length}" o_xyz="0 0 0" o_rpy="1.5707963 0 0" />
   </link>
   <joint name="rear_right_rack_wheel_joint" type="continuous">
